Commit message: create client interface for hand plugin
Working on an interface class for client applications to send commands to hand plugin running on gazebo server.

File: models/shadowhand.urdf (robot description, URDF)
Before this commit: robot shadowhand, 36 links, 35 joints
Joints:
- joint virtual_px_joint: limit lower=-0.5 upper=0.5 effort=5.0 velocity=5.0 -> lower=-1.0 upper=1.0 effort=25.0 velocity=25.0
- joint virtual_py_joint: limit lower=-0.5 upper=0.5 effort=5.0 velocity=5.0 -> lower=-1.0 upper=1.0 effort=25.0 velocity=25.0
- joint virtual_pz_joint: limit lower=0.0 upper=1.0 effort=20.0 velocity=20.0 -> lower=0.0 upper=1.0 effort=25.0 velocity=25.0
- joint virtual_rp_joint: limit lower=-1.57 upper=1.57 effort=10.01 velocity=0.0 -> lower=-1.57 upper=1.57 effort=25.0 velocity=25.0
- joint virtual_rr_joint: limit lower=-1.57 upper=1.57 effort=10.01 velocity=0.0 -> lower=-1.57 upper=1.57 effort=25.0 velocity=25.0
- joint virtual_ry_joint: limit lower=-1.57 upper=1.57 effort=10.01 velocity=0.0 -> lower=-1.57 upper=1.57 effort=25.0 velocity=25.0
