Commit message: add basic features to plugin

File: models/baxter_gripper.urdf (robot description, URDF)
Before this commit: robot baxter_gripper, 7 links, 6 joints
Links:
- removed link base
- added link hand
Joints:
- removed joint base_joint
- added joint gripper_base: type fixed, parent hand, child gripper_base, origin xyz=0 0 0.025 rpy=0 0 0

Commit message: fix floating gripper

File: models/baxter_gripper.urdf (robot description, URDF)
Before this commit: robot baxter_gripper, 7 links, 6 joints
Links:
- removed link hand
- added link world
Joints:
- removed joint gripper_base
- added joint virtual_prismatic_joint: type prismatic, parent world, child gripper_base, origin xyz=0 0 0 rpy=0 0 0, axis 0 0 1, limit lower=0.0 upper=0.5 effort=20.0 velocity=5.0

Commit message: add revolute joint

File: models/baxter_gripper.urdf (robot description, URDF)
Before this commit: robot baxter_gripper, 7 links, 6 joints
Links:
- added link virtual_link, mass 0.001; collision cylinder length=0.01 radius=0.01; visual cylinder length=0.01 radius=0.01
Joints:
- added joint virtual_revolute_joint: type revolute, parent virtual_link, child gripper_base, origin xyz=0 0 0 rpy=0 0 0, axis 0 0 1, limit lower=0.0 upper=3.5 effort=20.0 velocity=5.0
- joint virtual_prismatic_joint: child gripper_base -> virtual_link

Commit message: add virtual joints for 6 dof
Gripper can now move in unconstrained 3D space using 6 virtual joints.

File: models/baxter_gripper.urdf (robot description, URDF)
Before this commit: robot baxter_gripper, 8 links, 7 joints
Links:
- removed link virtual_link
- added link virtual_px_link, mass 0.001; collision cylinder length=0.001 radius=0.01; visual cylinder length=0.01 radius=0.01
- added link virtual_py_link, mass 0.001; collision cylinder length=0.001 radius=0.01; visual cylinder length=0.01 radius=0.01
- added link virtual_pz_link, mass 0.001; collision cylinder length=0.001 radius=0.01; visual cylinder length=0.01 radius=0.01
- added link virtual_rp_link, mass 0.001; collision cylinder length=0.001 radius=0.01; visual cylinder length=0.01 radius=0.01
- added link virtual_rr_link, mass 0.001; collision cylinder length=0.001 radius=0.01; visual cylinder length=0.01 radius=0.01
Joints:
- removed joint virtual_prismatic_joint
- removed joint virtual_revolute_joint
- added joint virtual_px_joint: type prismatic, parent world, child virtual_px_link, origin xyz=0 0 0 rpy=0 0 0, axis 1 0 0, limit lower=0.0 upper=0.5 effort=20.0 velocity=5.0
- added joint virtual_py_joint: type prismatic, parent virtual_px_link, child virtual_py_link, origin xyz=0 0 0 rpy=0 0 0, axis 0 1 0, limit lower=0.0 upper=0.5 effort=20.0 velocity=5.0
- added joint virtual_pz_joint: type prismatic, parent virtual_py_link, child virtual_pz_link, origin xyz=0 0 0 rpy=0 0 0, axis 0 0 1, limit lower=0.0 upper=0.5 effort=20.0 velocity=5.0
- added joint virtual_rp_joint: type continuous, parent virtual_rr_link, child virtual_rp_link, origin xyz=0 0 0 rpy=0 0 0, axis 0 1 0, limit effort=20.0 velocity=5.0
- added joint virtual_rr_joint: type continuous, parent virtual_pz_link, child virtual_rr_link, origin xyz=0 0 0 rpy=0 0 0, axis 1 0 0, limit effort=20.0 velocity=5.0
- added joint virtual_ry_joint: type continuous, parent virtual_rp_link, child gripper_base, origin xyz=0 0 0 rpy=0 0 0, axis 0 0 1, limit effort=20.0 velocity=5.0

Commit message: fix order of rpy operations

File: models/baxter_gripper.urdf (robot description, URDF)
Before this commit: robot baxter_gripper, 12 links, 11 joints
Joints:
- joint virtual_rr_joint: axis 1 0 0 -> 0 0 1
- joint virtual_ry_joint: axis 0 0 1 -> 1 0 0

Commit message: fix rpy coordinates in gripper urdf

File: models/baxter_gripper.urdf (robot description, URDF)
Before this commit: robot baxter_gripper, 12 links, 11 joints
Links:
- removed link virtual_rr_link
- added link virtual_ry_link, mass 0.001; collision cylinder length=0.001 radius=0.01; visual cylinder length=0.01 radius=0.01
Joints:
- joint virtual_rp_joint: parent virtual_rr_link -> virtual_ry_link
- joint virtual_rr_joint: axis 0 0 1 -> 1 0 0; child virtual_rr_link -> gripper_base; parent virtual_pz_link -> virtual_rp_link
- joint virtual_ry_joint: axis 1 0 0 -> 0 0 1; child gripper_base -> virtual_ry_link; parent virtual_rp_link -> virtual_pz_link

Commit message: able to lift box
Preliminary testing has shown that it's possible to grasp box using gripper, with fast simulation.

File: models/baxter_gripper.urdf (robot description, URDF)
Before this commit: robot baxter_gripper, 12 links, 11 joints
Joints:
- joint virtual_px_joint: limit lower=0.0 upper=0.5 effort=20.0 velocity=5.0 -> lower=0.0 upper=0.5 effort=40.0 velocity=5.0
- joint virtual_py_joint: limit lower=0.0 upper=0.5 effort=20.0 velocity=5.0 -> lower=0.0 upper=0.5 effort=40.0 velocity=5.0
- joint virtual_pz_joint: limit lower=0.0 upper=0.5 effort=20.0 velocity=5.0 -> lower=0.0 upper=0.5 effort=40.0 velocity=5.0
- joint virtual_rp_joint: limit effort=20.0 velocity=5.0 -> effort=40.0 velocity=5.0
- joint virtual_rr_joint: limit effort=20.0 velocity=5.0 -> effort=40.0 velocity=5.0
- joint virtual_ry_joint: limit effort=20.0 velocity=5.0 -> effort=40.0 velocity=5.0

Commit message: change velocity in msg. add grasp demo

File: models/baxter_gripper.urdf (robot description, URDF)
Before this commit: robot baxter_gripper, 12 links, 11 joints
Joints:
- joint gripper_r_finger_joint: mimic joint=gripper_l_finger_joint multiplier=-1.0 -> (none)

Commit message: remove gripper plugin; update baxter urdf
Removed unused and outdated gripper plugin.
Current hand plugin should work for grippers as well.

File: models/baxter_gripper.urdf (robot description, URDF)
Before this commit: robot baxter_gripper, 12 links, 11 joints
Links:
- link virtual_px_link: geometry collision cylinder length=0.001 radius=0.005; visual cylinder length=0.01 radius=0.005
- link virtual_py_link: geometry collision cylinder length=0.001 radius=0.005; visual cylinder length=0.01 radius=0.005
- link virtual_pz_link: geometry collision cylinder length=0.001 radius=0.005; visual cylinder length=0.01 radius=0.005
- link virtual_rp_link: geometry collision cylinder length=0.001 radius=0.005; visual cylinder length=0.01 radius=0.005
- link virtual_ry_link: geometry collision cylinder length=0.001 radius=0.005; visual cylinder length=0.01 radius=0.005
Joints:
- joint virtual_px_joint: limit lower=0.0 upper=0.5 effort=40.0 velocity=5.0 -> lower=-1.0 upper=1.0 effort=25.0 velocity=25.0
- joint virtual_py_joint: limit lower=0.0 upper=0.5 effort=40.0 velocity=5.0 -> lower=-1.0 upper=1.0 effort=25.0 velocity=25.0
- joint virtual_pz_joint: limit lower=0.0 upper=0.5 effort=40.0 velocity=5.0 -> lower=0.0 upper=1.0 effort=25.0 velocity=25.0
- joint virtual_rp_joint: limit effort=40.0 velocity=5.0 -> lower=-1.57 upper=1.57 effort=25.0 velocity=25.0; type continuous -> revolute
- joint virtual_rr_joint: limit effort=40.0 velocity=5.0 -> lower=-1.57 upper=1.57 effort=25.0 velocity=25.0; type continuous -> revolute
- joint virtual_ry_joint: limit effort=40.0 velocity=5.0 -> lower=-1.57 upper=1.57 effort=25.0 velocity=25.0; type continuous -> revolute

Commit message: tune virtual joints and pid parameters

File: models/baxter_gripper.urdf (robot description, URDF)
Before this commit: robot baxter_gripper, 12 links, 11 joints
Links:
- link virtual_px_link: mass 0.001 -> 01
- link virtual_py_link: mass 0.001 -> 01
- link virtual_pz_link: mass 0.001 -> 01
- link virtual_rp_link: mass 0.001 -> 01
- link virtual_ry_link: mass 0.001 -> 01
Joints:
- joint virtual_rp_joint: limit lower=-1.57 upper=1.57 effort=25.0 velocity=25.0 -> effort=25.0 velocity=25.0; type revolute -> continuous
- joint virtual_rr_joint: limit lower=-1.57 upper=1.57 effort=25.0 velocity=25.0 -> effort=25.0 velocity=25.0; type revolute -> continuous
- joint virtual_ry_joint: limit lower=-1.57 upper=1.57 effort=25.0 velocity=25.0 -> effort=25.0 velocity=25.0; type revolute -> continuous

Commit message: fix robot description files

File: models/baxter_gripper.urdf (robot description, URDF)
Before this commit: robot baxter_gripper, 12 links, 11 joints
Links:
- link virtual_px_link: mass 01 -> 1
- link virtual_py_link: mass 01 -> 1
- link virtual_pz_link: mass 01 -> 1
- link virtual_rp_link: mass 01 -> 1
- link virtual_ry_link: mass 01 -> 1

File: models/shadowhand.urdf (robot description, URDF)
Before this commit: robot shadowhand, 36 links, 35 joints
Links:
- link virtual_px_link: mass 0.001 -> 1
- link virtual_py_link: mass 0.001 -> 1
- link virtual_pz_link: mass 0.001 -> 1
- link virtual_rp_link: mass 0.001 -> 1
- link virtual_ry_link: mass 0.001 -> 1
Joints:
- joint virtual_rp_joint: limit lower=-1.57 upper=1.57 effort=25.0 velocity=25.0 -> effort=50.00 velocity=1.0; type revolute -> continuous
- joint virtual_rr_joint: limit lower=-1.57 upper=1.57 effort=25.0 velocity=25.0 -> effort=25.0 velocity=25.0; type revolute -> continuous
- joint virtual_ry_joint: limit lower=-1.57 upper=1.57 effort=25.0 velocity=25.0 -> effort=50.00 velocity=1.0; type revolute -> continuous
