Commit message: fix few issues
Testing grasping pipeline

File: models/baxter_standard_basic.urdf (robot description, URDF)
Before this commit: robot baxter_gripper, 12 links, 11 joints
Joints:
- joint gripper_l_finger_joint: limit lower=0.0 upper=0.020833 effort=20.0 velocity=5.0 -> lower=0.0 upper=0.028833 effort=100.0 velocity=5.0
- joint gripper_r_finger_joint: limit lower=-0.020833 upper=0.0 effort=20.0 velocity=5.0 -> lower=-0.028833 upper=0.0 effort=100.0 velocity=5.0
